File: hw/pwt-temp.kicad_pcb (KiCad board)
At the start: 0 parts

Commit message: Schaltplan Messplatine fertig
Parts:
- added C1: 100nF, 00_pwt-temp_lib:C_0603, F.Cu at (165.1, 83.8)
- added C10: 100n, 00_pwt-temp_lib:C_0603, F.Cu at (152.7, 98.4)
- added C11: 100n, 00_pwt-temp_lib:C_0603, F.Cu at (165.1, 88.4)
- added C12: 100n, 00_pwt-temp_lib:C_0603, F.Cu at (156.6, 95.7)
- added C13: 18p, 00_pwt-temp_lib:C_0603, F.Cu at (152.7, 100.7)
- added C14: 100nF, 00_pwt-temp_lib:C_0603, F.Cu at (160.5, 98.0)
- added C15: 100n, 00_pwt-temp_lib:C_0603, F.Cu at (169.0, 83.8)
- added C16: 100n, 00_pwt-temp_lib:C_0603, F.Cu at (129.0, 111.1)
- added C17: 100n, 00_pwt-temp_lib:C_0603, F.Cu at (172.9, 86.1)
- added C18: 1u, 00_pwt-temp_lib:C_0603, F.Cu at (147.7, 107.8)
- added C19: 100n, 00_pwt-temp_lib:C_0603, F.Cu at (165.1, 86.1)
- added C2: 1u, 00_pwt-temp_lib:C_0603, F.Cu at (132.9, 111.1)
- added C20: 1u, 00_pwt-temp_lib:C_0603, F.Cu at (169.0, 86.1)
- added C21: 100n, 00_pwt-temp_lib:C_0603, F.Cu at (172.9, 83.8)
- added C22: 10u, 00_pwt-temp_lib:C_0603, F.Cu at (147.7, 103.2)
- added C3: 1u, 00_pwt-temp_lib:C_0603, F.Cu at (152.7, 96.1)
- added C4: 100n, 00_pwt-temp_lib:C_0603, F.Cu at (142.9, 111.9)
- added C5: 100n, 00_pwt-temp_lib:C_0603, F.Cu at (142.9, 109.6)
- added C6: 1u, 00_pwt-temp_lib:C_0603, F.Cu at (163.6, 90.7)
- added C7: 1u, 00_pwt-temp_lib:C_0603, F.Cu at (156.6, 100.3)
- added C8: 18p, 00_pwt-temp_lib:C_0603, F.Cu at (147.7, 100.9)
- added C9: 100n, 00_pwt-temp_lib:C_0603, F.Cu at (167.5, 90.7)
- added D1: D_SCH_40V_0.25A, 00_pwt-temp_lib:SOD_323, F.Cu at (124.9, 111.4)
- added H1: MountingHole_Pad, MountingHole:MountingHole_3.2mm_M3_Pad_Via, F.Cu at (185.4, 109.2)
- added H2: MountingHole_Pad, MountingHole:MountingHole_3.2mm_M3_Pad_Via, F.Cu at (185.4, 101.3)
- added H3: MountingHole_Pad, MountingHole:MountingHole_3.2mm_M3_Pad_Via, F.Cu at (177.5, 109.2)
- added H4: MountingHole_Pad, MountingHole:MountingHole_3.2mm_M3_Pad_Via, F.Cu at (177.5, 101.3)
- added J1: CON_USB_B_MINI, 00_pwt-temp_lib:CON_USB_B_MINI, F.Cu at (137.4, 78.7)
- added J2: CON_PH_2.54MM_2x3_VERT, 00_pwt-temp_lib:CON_PH_2.54MM_2x3_VERT, F.Cu at (124.5, 73.7)
- added J3: CON_PH_2.54MM_2x3_VERT, 00_pwt-temp_lib:CON_PH_2.54MM_2x3_VERT, F.Cu at (152.4, 73.7)
- added R1: 10k, 00_pwt-temp_lib:R_0603, F.Cu at (169.0, 88.4)
- added R10: 20R, 00_pwt-temp_lib:R_0603, F.Cu at (156.6, 98.0)
- added R2: 27.4R, 00_pwt-temp_lib:R_0603, F.Cu at (147.7, 105.5)
- added R3: 27.4R, 00_pwt-temp_lib:R_0603, F.Cu at (151.6, 103.0)
- added R4: 1k, 00_pwt-temp_lib:R_0603, F.Cu at (156.6, 102.6)
- added R5: 1k, 00_pwt-temp_lib:R_0603, F.Cu at (164.4, 95.3)
- added R6: 10k, 00_pwt-temp_lib:R_0603, F.Cu at (146.8, 110.1)
- added R7: 10k, 00_pwt-temp_lib:R_0603, F.Cu at (151.6, 105.3)
- added R8: 10k, 00_pwt-temp_lib:R_0603, F.Cu at (163.6, 93.0)
- added R9: 10k, 00_pwt-temp_lib:R_0603, F.Cu at (160.5, 95.7)
- added S1: MECH_BTN_SMD_SMALL, 00_pwt-temp_lib:MECH_BTN_SMD_SMALL, F.Cu at (158.1, 92.2)
- added U1: PMIC_LDO_3V3_0.2A, 00_pwt-temp_lib:SOT_23_3, F.Cu at (148.3, 97.5)
- added U2: IC_W25Q16JV, 00_pwt-temp_lib:IC_W25Q16JV, F.Cu at (165.1, 73.7)
- added U3: IC_RP2040, 00_pwt-temp_lib:IC_RP2040, F.Cu at (141.1, 103.8)
- added U4: IC_AMG8834, 00_pwt-temp_lib:IC_AMG8834, F.Cu at (129.6, 104.2)
- added Y1: OSC_ABM10-12.000MHZ, 00_pwt-temp_lib:OSC_ABM10, F.Cu at (138.7, 110.4)
Other:
- copper layers 0 -> 2
