File: hw/pcb_mess/pwt-temp_pcb_mess.kicad_pcb (KiCad board)
At the start: 2 copper layers, 46 parts, among them J1 CON_USB_B_MINI, J2 PinHeader_2x03_P2.54mm_Vertic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, J3 PinHeader_2x03_P2.54mm_Vertic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, U1 PMIC_LDO_3V3_0.2A, U2 SOIC_8, U3 IC_RP2040, U4 IC_AMG8834, Y1 OSC_ABM10-12.000MHZ

Commit message: Finished Layout
Parts:
- added S2: MECH_SW_DIP4_SMD, 00_pwt-temp_lib:MECH_SW_DIP4_SMD, F.Cu at (157.5, 91.7)
- moved C21 117.2 mm to (105.9, 78.5), turned to -90 degrees
- moved H1 92.5 mm to (115.5, 67.5)
- moved R9 89.3 mm to (132.4, 72.7), turned to -90 degrees
- moved U1 80.3 mm to (138.6, 94.8), turned to -90 degrees
- moved R8 76.6 mm to (133.9, 72.7), turned to -90 degrees
- moved H2 76.2 mm to (115.5, 92.5)
- moved C15 73.8 mm to (138.6, 91.8)
- moved C14 70.2 mm to (141.3, 94.8), turned to 90 degrees
- moved R3 69.4 mm to (153.4, 71.6), turned to -90 degrees
- moved R10 66.1 mm to (131.5, 85.7)
- moved R7 65.5 mm to (135.4, 72.7), turned to -90 degrees
- moved C18 63.0 mm to (137.8, 85.7)
- moved R2 62.4 mm to (151.9, 71.6), turned to -90 degrees
- moved R6 61.9 mm to (153.4, 87.3), turned to 90 degrees
- moved C20 61.5 mm to (131.5, 87.2)
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Connections:
- U3 pad 24: unconnected-(U3-SWCLK) -> /SWCLK
- U3 pad 25: unconnected-(U3-SWDIO) -> /SWDIO
Routing:
- net /~{BOOT}: track 0.00 -> 23.0 mm
- net /I2C_INT_INT: track 0.00 -> 19.6 mm
- net /I2C_INT_SCL: track 0.00 -> 18.2 mm
- net /I2C_INT_SDA: track 0.00 -> 16.6 mm
- net +3V3: track 29.1 -> 42.4 mm, vias 8 -> 15
- net GND: track 17.3 -> 27.9 mm, vias 13 -> 30
- net /SPI_~{CS}: track 29.9 -> 22.3 mm
- net /SPI_SD1: track 23.5 -> 16.7 mm
- net /SWCLK: track 0.00 -> 5.77 mm
- net /SWDIO: track 0.00 -> 5.57 mm
- net /SPI_SD0: track 11.4 -> 6.62 mm
- net /DVDD: track 0.00 -> 4.44 mm
- net Net-(U3-RUN): track 0.76 -> 4.30 mm
- net /SPI_SD2: track 18.3 -> 15.1 mm
- net /AVDD: track 0.00 -> 2.65 mm
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Other:
- board outline added: 60 x 35 mm
