File: hw/pcb_mess/pwt-temp_pcb_mess.kicad_pcb (KiCad board)
At the start: 2 copper layers, 60 x 35 mm, 47 parts, among them J1 CON_USB_B_MINI, J2 PinHeader_2x03_P2.54mm_Vertic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, J3 PinHeader_2x03_P2.54mm_Vertic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, U1 PMIC_LDO_3V3_0.2A, U2 SOIC_8, U3 IC_RP2040, U4 IC_AMG8834, Y1 OSC_ABM10-12.000MHZ

Commit message: Layout fertiggestellt
Parts:
- J2, J3: value PinHeader_2x03_P2.54mm_Vertical -> CON_PH_2.54MM_2x3_VERT
- U2: value SOIC_8 -> IC_W25Q16JV
- moved C19 51.4 mm to (159.2, 79.3), turned to -90 degrees
- moved C22 45.6 mm to (127.8, 83.2), turned to 180 degrees
- moved C21 15.2 mm to (120.9, 76.2)
- moved S2 5.28 mm to (156.6, 86.5)
- moved J1 3.40 mm to (125.5, 96.1)
- moved C17 2.73 mm to (144.7, 87.5)
- moved Y1 2.73 mm to (144.7, 85.0)
- moved C12 2.73 mm to (149.9, 84.8)
- moved C16 2.73 mm to (142.5, 84.8)
- moved C3 2.73 mm to (148.4, 84.8)
- moved R5 2.73 mm to (146.9, 84.8)
- moved R6 2.73 mm to (152.3, 84.8)
- moved C1 2.55 mm to (142.5, 74.1)
- moved C10 2.55 mm to (149.9, 69.1)
- moved C11 2.55 mm to (153.3, 72.1)
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Connections:
- U3 pad 29: unconnected-(U3-GPIO18) -> /ADDR_3
- U3 pad 30: unconnected-(U3-GPIO19) -> /ADDR_2
- U3 pad 31: unconnected-(U3-GPIO20) -> /ADDR_1
- U3 pad 32: unconnected-(U3-GPIO21) -> /ADDR_0
Routing:
- net /I2C_EXT_SDA: track 0.00 -> 91.8 mm, vias 0 -> 1
- net /I2C_EXT_SCL: track 0.00 -> 65.2 mm, vias 0 -> 1
- net /USB_DN: track 1.02 -> 49.2 mm, vias 1 -> 2
- net /USB_DP: track 1.02 -> 46.9 mm, vias 1 -> 2
- net GND: track 27.9 -> 61.3 mm, vias 30 -> 36
- net +3V3: track 42.4 -> 72.8 mm, vias 15 -> 19
- net /VBUS: track 0.00 -> 14.5 mm
- net /ADDR_0: track 0.00 -> 8.32 mm
- net /ADDR_1: track 0.00 -> 6.87 mm
- net Net-(D1-K): track 0.00 -> 5.81 mm
- net /ADDR_2: track 0.00 -> 5.44 mm
- net /ADDR_3: track 0.00 -> 3.97 mm
- net /VCORE: track 11.9 -> 14.5 mm, vias 0 -> 3
- net Net-(U3-RUN): track 4.30 -> 3.64 mm
- net Net-(U3-XIN): track 7.70 -> 8.28 mm
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- added copper zone on In2.Cu, net +3V3
- added copper zone on In2.Cu, net /VCORE
- added copper zone on B.Cu, net GND
- added copper zone on In1.Cu, net GND
Other:
- copper layers 2 -> 4

Commit message: Added rendering
Parts:
- added TP1: TestPoint, TestPoint:TestPoint_Pad_D1.5mm, B.Cu at (151.0, 90.0)
- added TP2: TestPoint, TestPoint:TestPoint_Pad_D1.5mm, B.Cu at (148.0, 90.0)
- added TP3: TestPoint, TestPoint:TestPoint_Pad_D1.5mm, B.Cu at (145.0, 90.0)
- added TP4: TestPoint, TestPoint:TestPoint_Pad_D1.5mm, B.Cu at (142.0, 90.0)
- moved S1 2.04 mm to (130.5, 63.8)
Connections:
- net Net-(U3-RUN) renamed /NRST
Routing:
- net /SWCLK: track 5.52 -> 14.4 mm, vias 0 -> 1
- net /NRST: track 3.64 -> 12.0 mm, vias 0 -> 1
- net /SWDIO: track 5.32 -> 11.9 mm, vias 0 -> 1
- net /~{BOOT}: track 23.0 -> 27.9 mm
- net GND: track 61.3 -> 64.4 mm, vias 36 -> 40
- net +3V3: track 72.8 -> 73.9 mm, vias 19 -> 20
Other:
- board text added: "GND"
- board text added: "NRST"
- board text added: "SWCLK"
- board text added: "SWDIO"
