File: hw/pcb_mess/pwt-temp_pcb_mess.kicad_sch (KiCad schematic)
At the start: 46 parts, among them J1 CON_USB_B_MINI, J2 CON_PH_2.54MM_2x3_VERT, J3 CON_PH_2.54MM_2x3_VERT, U1 PMIC_LDO_3V3_0.2A, U2 IC_W25Q16JV, U3 IC_RP2040, U4 IC_AMG8834, Y1 OSC_ABM10-12.000MHZ

Commit message: Layout & Schaltplan erzeugt
Parts:
- renumbered C4 to C1, C16 to C10, C7 to C11, C17 to C13, C2 to C14, C3 to C15, C8 to C16, C13 to C17, C9 to C2, C14 to C3, C5 to C4, C10 to C5, C1 to C6, C15 to C7, C6 to C8, C11 to C9

Commit message: Finished Layout
Parts:
- added S2: MECH_SW_DIP4_SMD, 00_pwt-temp_lib:MECH_SW_DIP4_SMD, symbol 00_pwt-temp_lib:MECH_SW_DIP4_SMD
Connections:
- net GND: now also S2.5, S2.6, S2.7, S2.8
- net SWCLK: now reaches U3.24 (SWCLK)
- net SWDIO: now reaches U3.25 (SWDIO)
- new net ADDR_0: S2.1
- new net ADDR_1: S2.2
- new net ADDR_2: S2.3
- new net ADDR_3: S2.4
- no-connect marks 4 -> 2
Other:
- moved on the sheet: C16, C17, C19, C21, J2, J3, R5, Y1

Commit message: Layout fertiggestellt
Connections:
- net ADDR_0: now also U3.32 (GPIO21)
- net ADDR_1: now also U3.31 (GPIO20)
- net ADDR_2: now also U3.30 (GPIO19)
- net ADDR_3: now also U3.29 (GPIO18)
Other:
- moved on the sheet: S2

Commit message: Added rendering
Parts:
- added TP1, TP2, TP3, TP4: TestPoint, TestPoint:TestPoint_Pad_D1.5mm, symbol Connector:TestPoint
Connections:
- net GND: now also TP4.1
- net SWCLK: now also TP3.1
- net SWDIO: now also TP2.1
- net NRST: now reaches R6.2, U3.26 (RUN)
- net NRST: now also TP1.1
Other:
- moved on the sheet: H1, H2, H3, H4, R6
